File: LED-test-board-v0.1.kicad_pcb (KiCad board)
At the start: 2 copper layers, 76 x 50.8 mm, 259 parts, among them P1 CONN_01X01, P10 CONN_01X01, P100 CONN_01X01, P101 CONN_01X01, P102 CONN_01X01, P103 CONN_01X01, P104 CONN_01X01, P105 CONN_01X01, P106 CONN_01X01, P107 CONN_01X01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

Commit message: Fix net-name error and remove unnecessary library
Connections:
- net LED_ANODE renamed LED_CATHODE
